File: pcb/capstone_pcb.kicad_sch (KiCad schematic)
At the start: 46 parts, among them IC6 BSS138, Q1 BSS138, U2 BMI270, U3 NRF52840-QIAA-R, U4 MAX30102EFD+T, X1 32MHz, X2 32.768kHz

Commit message: Add files via upload
Parts:
- removed B1: CR-2032/VCN, BAT_CR-2032_PAN, symbol 2026-03-01_23-35-29:CR-2032_VCN
- added BT1: Battery_Cell, Battery:BatteryHolder_Keystone_1058_1x2032, symbol Device:Battery_Cell
- C1, C11, C12, C14, C15, C16, C17, C18, C19, C2, C20, C21, C23, C24, C25, C26, C27, C3, C4, C5, C6, C7, C8, C9: footprint (none) -> Capacitor_SMD:C_0201_0603Metric
- L1: footprint (none) -> Inductor_SMD:L_0201_0603Metric
- R1, R2, R3, R4, R5, R6: footprint (none) -> Resistor_SMD:R_0201_0603Metric
- R7: renamed from R2; footprint (none) -> Resistor_SMD:R_0201_0603Metric
- U2: footprint BMI270:XDCR_BMI270 -> bmi270:XDCR_BMI270
- U3: footprint AQFN73_7X7_NOR -> Library:nrf52840_qiaa_r
- U4: footprint 21-1048_F143A5+1_MXM -> MAX30102EFD_T:XDCR_MAX30101EFD_
- X1, X2: footprint (none) -> Crystal:Crystal_SMD_3215-2Pin_3.2x1.5mm
- gave numbers to parts that had none: 1
Connections:
- net Earth: now also BT1.2 (-)
- net VBAT: now also BT1.1 (+)
- no-connect marks 0 -> 51
Other:
- moved on the sheet: C5
