File: capstone_pcb/capstone_pcb.kicad_pcb (KiCad board)
At the start: 4 copper layers, 76.2 x 57.2 mm, 45 parts, among them IC6 BSS138, P1 MHDR1X5, Q1 BSS138, U1 AMS1117-3.3, U2 BMI270, U3 NRF52840-QIAA-R, U4 MAX30102EFD+T, U5 AMS1117-1.8, X1 32MHz, X2 32.768kHz

Commit message: update pcb
Parts:
- C1, C11, C15, C16, C17, C18, C2, C24, C25, C27, C3, C4, C5, C6, C7, C8, C9: footprint Capacitor_SMD:C_0201_0603Metric -> Capacitor_SMD:C_0402_1005Metric
- L1: footprint Inductor_SMD:L_0201_0603Metric -> Inductor_SMD:L_0402_1005Metric
- R1, R2, R3, R4, R6: footprint Resistor_SMD:R_0201_0603Metric -> Resistor_SMD:R_0402_1005Metric
- moved C24 20.1 mm to (87.0, 68.7), turned to 90 degrees
- moved C6 13.5 mm to (85.2, 68.7), turned to 90 degrees
- moved C8 8.46 mm to (106.0, 69.5), turned to 90 degrees
- moved C15 6.96 mm to (127.9, 51.1)
- moved C16 6.22 mm to (104.3, 69.5), turned to 90 degrees
- moved R4 0.25 mm to (115.2, 41.7)
Routing:
- net +1.8V: track 67.7 -> 97.5 mm
- net /SDA: track 5.34 -> 34.5 mm, vias 0 -> 2
- net +5V: track 94.0 -> 79.8 mm, vias 5 -> 6
- net Earth: track 122.0 -> 109.8 mm, vias 22 -> 23
- net /DEC4 6: track 9.16 -> 2.46 mm
- net +3.3V: track 124.2 -> 121.9 mm, vias 10 -> 11
- net Net-(U3-P0.01/XL2): track 15.4 -> 16.6 mm
- net Net-(U3-ANT): track 9.65 -> 8.73 mm
- net /BSCL: track 11.1 -> 11.7 mm
- net /SCL: track 30.8 -> 31.2 mm, vias 0 -> 2

Commit message: update pcb
Parts:
- moved C14 5.08 mm to (126.7, 67.3)
- moved C21 2.54 mm to (126.7, 66.0)
- moved R5 1.31 mm to (122.0, 34.9), turned to -90 degrees
- moved R4 1.31 mm to (114.0, 41.0), turned to 180 degrees
- moved C17 0.34 mm to (115.6, 63.5), turned to 90 degrees
- turned C18 to 90 degrees
Routing:
- net Earth: track 109.8 -> 89.3 mm, vias 23 -> 24
- net +3.3V: track 121.9 -> 109.2 mm, vias 11 -> 10
- net /ASDA: track 16.5 -> 14.7 mm
- net Net-(U3-P0.01/XL2): track 16.6 -> 15.4 mm
- net /BSCL: track 11.7 -> 10.7 mm
- net +5V: track 79.8 -> 80.1 mm, vias 6 -> 7

Commit message: update pcb
Routing:
- net +3.3V: track 109.2 -> 110.4 mm
Changed lines of the file:
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@@
   (segment (start 106.045 70.993) (end 106.172 71.12) (width 0.25) (layer "F.Cu") (net 16))
   (segment (start 126.175 66.04) (end 126.175 64.77) (width 0.25) (layer "F.Cu") (net 16))
+  (segment (start 105.09 43.18) (end 102.87 43.18) (width 0.25) (layer "F.Cu") (net 16))
   (segment (start 120.65 31.75) (end 119.38 30.48) (width 0.25) (layer "F.Cu") (net 16))
   (segment (start 121.285 57.15) (end 120.777 56.642) (width 0.25) (layer "F.Cu") (net 16))
@@
   (segment (start 80.67 50.8) (end 86.97 50.8) (width 0.25) (layer "F.Cu") (net 16))
   (segment (start 104.14 50.8) (end 104.775 50.8) (width 0.25) (layer "F.Cu") (net 16))
-  (segment (start 105.09 43.18) (end 104.14 43.18) (width 0.25) (layer "F.Cu") (net 16))
   (segment (start 106.045 52.07) (end 106.045 54.58) (width 0.25) (layer "F.Cu") (net 16))
   (segment (start 98.9525 60.7975) (end 99.27462 60.7975) (width 0.25) (layer "F.Cu") (net 16))
@@
   (via (at 106.172 71.12) (size 0.8) (drill 0.4) (layers "F.Cu" "B.Cu") (net 16))
   (via (at 125.73 63.5) (size 0.8) (drill 0.4) (layers "F.Cu" "B.Cu") (net 16))
-  (via (at 104.14 43.18) (size 0.8) (drill 0.4) (layers "F.Cu" "B.Cu") (net 16))
+  (via (at 102.87 43.18) (size 0.8) (drill 0.4) (layers "F.Cu" "B.Cu") (net 16))
   (via (at 120.777 56.642) (size 0.8) (drill 0.4) (layers "F.Cu" "B.Cu") (net 16))
   (via (at 122.682 52.07) (size 0.8) (drill 0.4) (layers "F.Cu" "B.Cu") (net 16))

Commit message: update pcb
Parts:
- moved IC6 6.35 mm to (121.9, 44.5), turned to 180 degrees
- moved C26 2.55 mm to (106.2, 52.1)
- moved C25 0.13 mm to (106.2, 54.6)
Routing:
- net +3.3V: track 110.4 -> 78.4 mm, vias 10 -> 5
- net +1.8V: track 97.7 -> 88.3 mm, vias 5 -> 3
- net /BSDA: track 18.7 -> 9.92 mm
- net /ASDA: track 14.7 -> 12.0 mm
